File: LED_drv.brd (EAGLE design)
At the start: 160 x 100 mm, 103 parts, among them IC1 LM3409, IC2 LM393D, Q2 IPD50R380, T1 IRLR9343PBF, T2 BCX56, T4 BT169, T5 BT169, T6 TLP266J

Commit message: screenshot added
minor updates and comments
Parts:
- removed C13: 22uF/50V, rcl:E5-6
- removed PAD21: (no value), wirepad:SMD1,27-2,54
- added IC3: (no value), TI:SOT23-3
- added R41: 100k, rcl:R1206
- added T3: BC847, transistor:SOT23
- added T7: IPD50R380, miscrel:TO252-3-11
- C3: value 22uF/50V -> 47uF/50V
- C5: value 470p/50V -> 1n/50V; device rcl:C1206 -> rcl:C0603
- D10: value 1n4002 -> 20V; device diode:DO214AC -> diode:SOD80C
- D11: value 1n4002 -> 18V; device diode:DO214AC -> diode:SOD80C
- L1: value CDRH104R -> 68uH
- R28: value 1M -> 47k
- R39: value 86k -> 22k
- R4, R5: value 1R -> 0.4R
- R40: value 47k -> 20k; device rcl:R0805 -> rcl:R1206
- R6: value 470k -> 100k
- R7: value 15k -> 12k
- moved D11 69.5 mm to (-27.9, -74.9)
- moved D10 50.2 mm to (-5.08, -53.3)
- moved R40 18.4 mm to (-5.08, -47.0)
- moved R39 18.4 mm to (-5.08, -40.6)
- moved R7 2.44 mm to (45.5, 45.5)
- moved C5 2.42 mm to (45.2, 47.1)
Connections:
- removed net N$41: D10.A, D11.C
- removed net N$44: D11.A, R38.1, R39.2
- new net GNDA: C7.2, C9.-, D11.A, D4.A, D6.A, IC2.4, PAD10.1, R23.2, R40.1, R9.2, T3.2, T7.3
- new net N$42: D10.A, T3.1
- new net N$43: IC3.1, IC3.2, PAD14.1, R38.1, R6.3
- net GND: now also C2.2, IC3.3, T7.2; no longer C13.-, C2.1, C7.2, C9.-, D10.C, D4.A, D6.A, IC2.4, PAD10.1, PAD21.1, R23.2, R9.2
- net N$11: no longer C13.+
- net N$2: now also D11.C, R41.1, T3.3, T7.1; no longer C12.+, IC1.10, IC1.8, PAD12.1, PAD20.1, R2.2, R38.2, R4.2, R5.2, S1.2
- net N$40: now also D10.C, R40.2; no longer PAD14.1, R6.3
- net N$5: now also C2.1; no longer C2.2
- net V+: now also C12.+, IC1.10, IC1.8, PAD12.1, PAD20.1, R2.2, R38.2, R39.2, R4.2, R41.2, R5.2, S1.2
Routing:
- net N$2: track 64.0 -> 0.00 mm
- net ACTIVATION: track 55.7 -> 17.1 mm
- net N$10: track 33.4 -> 0.00 mm
- net GND: track 36.9 -> 6.49 mm
- net N$8: track 20.5 -> 0.00 mm
- net N$4: track 19.2 -> 0.00 mm
- net N$5: track 18.8 -> 0.00 mm
- net N$9: track 18.2 -> 0.00 mm
- net N$11: track 13.3 -> 0.00 mm
- net N$6: track 11.9 -> 0.00 mm
- net N$1: track 11.4 -> 0.00 mm
- net N$13: track 6.33 -> 0.00 mm
- net N$3: track 2.83 -> 0.00 mm
- net N$37: track 2.77 -> 0.00 mm
- net N$36: track 2.77 -> 0.00 mm
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