File: LED_drv.sch (EAGLE design)
At the start: 98 parts, among them IC1 LM3409, IC2 LM393D, Q2 IPD50R380, T1 IRLR9343PBF, T2 BCX56, T4 BT169, T5 BT169, T6 TLP266J

Commit message: test_release
Parts:
- added D10, D11: 1n4002, diode:DIODE-DO214AC
- added R38: 51k, rcl:R-EU_R1206
- added R39: 86k, rcl:R-EU_R1206
- added R40: 47k, rcl:R-EU_R0805
- 0R: value 1R -> 0R
- R1: value (none) -> 7k5
- R2: value (none) -> 51k
Connections:
- new net N$40: PAD14.P, R39.1, R6.E
- new net N$41: D10.A, D11.C
- new net N$44: D11.A, R38.1, R39.2
- net GND: now also D10.C
- net N$2: now also R38.2; no longer PAD14.P, R6.E
Other:
- note added: "powinno byc max 47k"
- moved on the sheet: 0R, PAD12, PAD13, PAD17, S1
Changed lines of the file:
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@@
 <parts>
 <part name="IC1" library="TI" deviceset="LM3409" device=""/>
-<part name="R1" library="rcl" deviceset="R-EU_" device="R1206"/>
-<part name="R2" library="rcl" deviceset="R-EU_" device="R1206"/>
+<part name="R1" library="rcl" deviceset="R-EU_" device="R1206" value="7k5"/>
+<part name="R2" library="rcl" deviceset="R-EU_" device="R1206" value="51k"/>
 <part name="GND1" library="supply1" deviceset="GND" device=""/>
 <part name="GND2" library="supply1" deviceset="GND" device=""/>
@@
 <part name="C12" library="rcl" deviceset="CPOL-EU" device="E5-6" value="22uF/50V"/>
 <part name="C13" library="rcl" deviceset="CPOL-EU" device="E5-6" value="22uF/50V"/>
-<part name="0R" library="resistor" deviceset="R-EU_" device="R1206" value="1R"/>
+<part name="0R" library="resistor" deviceset="R-EU_" device="R1206" value="0R"/>
 <part name="R37" library="varistor" deviceset="S14K275_SMD" device=""/>
 <part name="F1" library="fuse" deviceset="SH22,5A" device=""/>
+<part name="D10" library="diode" deviceset="DIODE-" device="DO214AC" value="1n4002"/>
+<part name="D11" library="diode" deviceset="DIODE-" device="DO214AC" value="1n4002"/>
+<part name="R38" library="rcl" deviceset="R-EU_" device="R1206" value="51k"/>
+<part name="R39" library="rcl" deviceset="R-EU_" device="R1206" value="86k"/>
+<part name="R40" library="rcl" deviceset="R-EU_" device="R0805" value="47k"/>
 </parts>
 <sheets>
@@
 <text x="309.88" y="38.1" size="1.778" layer="91">podlacz do zasilacza w srodku</text>
 <text x="243.84" y="-35.56" size="1.778" layer="97">active high</text>
-<text x="-25.4" y="58.42" size="1.27" layer="97">TO Vcc !!!!</text>
+<text x="-38.1" y="58.42" size="1.27" layer="97">TO Vcc !!!!</text>
 <text x="-12.7" y="15.24" size="1.27" layer="91">pulldown</text>
+<text x="-30.48" y="-15.24" size="1.778" layer="91">powinno byc max 47k</text>
 </plain>
 <instances>
@@
 <instance part="R6" gate="G$1" x="-17.78" y="30.48"/>
 <instance part="GND7" gate="1" x="-17.78" y="20.32"/>
-<instance part="S1" gate="G$1" x="-25.4" y="33.02"/>
+<instance part="S1" gate="G$1" x="-38.1" y="33.02"/>
 <instance part="C5" gate="G$1" x="10.16" y="0"/>
 <instance part="R7" gate="G$1" x="2.54" y="-2.54" rot="R270"/>
@@
 <instance part="PAD11" gate="1" x="241.3" y="-53.34" rot="R90"/>
 <instance part="R32" gate="G$1" x="241.3" y="-40.64" rot="R270"/>
-<instance part="PAD12" gate="1" x="-27.94" y="40.64"/>
-<instance part="PAD13" gate="1" x="-27.94" y="7.62"/>
+<instance part="PAD12" gate="1" x="-40.64" y="40.64"/>
+<instance part="PAD13" gate="1" x="-40.64" y="7.62"/>
 <instance part="PAD14" gate="1" x="-15.24" y="38.1" rot="R180"/>
 <instance part="PAD15" gate="1" x="-15.24" y="25.4" rot="R180"/>
 <instance part="PAD16" gate="1" x="-10.16" y="33.02" rot="R270"/>
-<instance part="PAD17" gate="1" x="-27.94" y="22.86"/>
+<instance part="PAD17" gate="1" x="-40.64" y="22.86"/>
 <instance part="PAD18" gate="1" x="114.3" y="-2.54" rot="R180"/>
 <instance part="PAD19" gate="1" x="83.82" y="-17.78" rot="R180"/>
@@
 <instance part="C12" gate="G$1" x="81.28" y="33.02"/>
 <instance part="C13" gate="G$1" x="76.2" y="-12.7"/>
-<instance part="0R" gate="G$1" x="-25.4" y="15.24" rot="R90"/>
+<instance part="0R" gate="G$1" x="-38.1" y="15.24" rot="R90"/>
 <instance part="R37" gate="G$1" x="462.28" y="-15.24" rot="R90"/>
 <instance part="F1" gate="1" x="490.22" y="-38.1"/>
+<instance part="D10" gate="G$1" x="-27.94" y="27.94" rot="MR270"/>
+<instance part="D11" gate="G$1" x="-27.94" y="35.56" rot="MR270"/>
+<instance part="R38" gate="G$1" x="-27.94" y="45.72" rot="R90"/>
+<instance part="R39" gate="G$1" x="-22.86" y="38.1" rot="R180"/>
+<instance part="R40" gate="G$1" x="-17.78" y="-2.54" rot="R90"/>
 </instances>
 <busses>
@@
 <wire x1="55.88" y1="27.94" x2="50.8" y2="27.94" width="0.1524" layer="91"/>
 <wire x1="50.8" y1="35.56" x2="81.28" y2="35.56" width="0.1524" layer="91"/>
-<pinref part="R6" gate="G$1" pin="E"/>
-<wire x1="-17.78" y1="35.56" x2="-17.78" y2="38.1" width="0.1524" layer="91"/>
-<wire x1="-17.78" y1="38.1" x2="-17.78" y2="55.88" width="0.1524" layer="91"/>
-<wire x1="-17.78" y1="55.88" x2="50.8" y2="55.88" width="0.1524" layer="91"/>
+<wire x1="-38.1" y1="55.88" x2="-27.94" y2="55.88" width="0.1524" layer="91"/>
+<wire x1="-27.94" y1="55.88" x2="50.8" y2="55.88" width="0.1524" layer="91"/>
 <wire x1="50.8" y1="55.88" x2="50.8" y2="45.72" width="0.1524" layer="91"/>
 <wire x1="50.8" y1="55.88" x2="50.8" y2="58.42" width="0.1524" layer="91"/>
 <junction x="50.8" y="55.88"/>
 <pinref part="S1" gate="G$1" pin="S"/>
-<wire x1="-25.4" y1="38.1" x2="-25.4" y2="40.64" width="0.1524" layer="91"/>
-<wire x1="-25.4" y1="40.64" x2="-25.4" y2="55.88" width="0.1524" layer="91"/>
-<wire x1="-25.4" y1="55.88" x2="-17.78" y2="55.88" width="0.1524" layer="91"/>
-<junction x="-17.78" y="55.88"/>
+<wire x1="-38.1" y1="38.1" x2="-38.1" y2="40.64" width="0.1524" layer="91"/>
+<wire x1="-38.1" y1="40.64" x2="-38.1" y2="55.88" width="0.1524" layer="91"/>
 <pinref part="PAD12" gate="1" pin="P"/>
-<junction x="-25.4" y="40.64"/>
-<pinref part="PAD14" gate="1" pin="P"/>
-<junction x="-17.78" y="38.1"/>
+<junction x="-38.1" y="40.64"/>
 <pinref part="PAD20" gate="1" pin="P"/>
 <pinref part="C12" gate="G$1" pin="+"/>
+<pinref part="R38" gate="G$1" pin="2"/>
+<wire x1="-27.94" y1="50.8" x2="-27.94" y2="55.88" width="0.1524" layer="91"/>
+<junction x="-27.94" y="55.88"/>
 </segment>
 </net>
@@
 <junction x="-17.78" y="25.4"/>
 <wire x1="-17.78" y1="25.4" x2="-17.78" y2="22.86" width="0.1524" layer="91"/>
+<pinref part="D10" gate="G$1" pin="C"/>
+<wire x1="-27.94" y1="25.4" x2="-27.94" y2="22.86" width="0.1524" layer="91"/>
+<wire x1="-27.94" y1="22.86" x2="-17.78" y2="22.86" width="0.1524" layer="91"/>
+<junction x="-17.78" y="22.86"/>
 </segment>
 <segment>
@@
 <wire x1="7.62" y1="25.4" x2="7.62" y2="12.7" width="0.1524" layer="91"/>
 <wire x1="7.62" y1="12.7" x2="-10.16" y2="5.08" width="0.1524" layer="91"/>
-<wire x1="-10.16" y1="5.08" x2="-25.4" y2="5.08" width="0.1524" layer="91"/>
-<wire x1="-25.4" y1="5.08" x2="-25.4" y2="7.62" width="0.1524" layer="91"/>
-<label x="-25.4" y="5.08" size="1.27" layer="95" rot="R180" xref="yes"/>
+<wire x1="-10.16" y1="5.08" x2="-38.1" y2="5.08" width="0.1524" layer="91"/>
+<wire x1="-38.1" y1="5.08" x2="-38.1" y2="7.62" width="0.1524" layer="91"/>
+<label x="-38.1" y="5.08" size="1.27" layer="95" rot="R180" xref="yes"/>
 <pinref part="R28" gate="G$1" pin="2"/>
 <junction x="-10.16" y="5.08"/>
 <pinref part="PAD13" gate="1" pin="P"/>
-<wire x1="-25.4" y1="7.62" x2="-25.4" y2="10.16" width="0.1524" layer="91"/>
-<junction x="-25.4" y="7.62"/>
+<wire x1="-38.1" y1="7.62" x2="-38.1" y2="10.16" width="0.1524" layer="91"/>
+<junction x="-38.1" y="7.62"/>
 <pinref part="0R" gate="G$1" pin="1"/>
 </segment>
@@
 <pinref part="PAD17" gate="1" pin="P"/>
 <pinref part="0R" gate="G$1" pin="2"/>
-<wire x1="-25.4" y1="20.32" x2="-25.4" y2="22.86" width="0.1524" layer="91"/>
-<junction x="-25.4" y="22.86"/>
-<wire x1="-25.4" y1="22.86" x2="-25.4" y2="27.94" width="0.1524" layer="91"/>
+<wire x1="-38.1" y1="20.32" x2="-38.1" y2="22.86" width="0.1524" layer="91"/>
+<junction x="-38.1" y="22.86"/>
+<wire x1="-38.1" y1="22.86" x2="-38.1" y2="27.94" width="0.1524" layer="91"/>
 </segment>
 </net>
@@
 </segment>
 </net>
+<net name="N$40" class="0">
+<segment>
+<pinref part="PAD14" gate="1" pin="P"/>
+<pinref part="R6" gate="G$1" pin="E"/>
+<wire x1="-17.78" y1="35.56" x2="-17.78" y2="38.1" width="0.1524" layer="91"/>
+<junction x="-17.78" y="38.1"/>
+<pinref part="R39" gate="G$1" pin="1"/>
+</segment>
+</net>
+<net name="N$41" class="0">
+<segment>
+<pinref part="D10" gate="G$1" pin="A"/>
+<pinref part="D11" gate="G$1" pin="C"/>
+<wire x1="-27.94" y1="30.48" x2="-27.94" y2="33.02" width="0.1524" layer="91"/>
+</segment>
+</net>
+<net name="N$44" class="0">
+<segment>
+<pinref part="D11" gate="G$1" pin="A"/>
+<pinref part="R38" gate="G$1" pin="1"/>
+<wire x1="-27.94" y1="40.64" x2="-27.94" y2="38.1" width="0.1524" layer="91"/>
+<junction x="-27.94" y="38.1"/>
+<pinref part="R39" gate="G$1" pin="2"/>
+</segment>
+</net>

Commit message: screenshot added
minor updates and comments
Parts:
- removed C13: 22uF/50V, rcl:CPOL-EUE5-6
- removed PAD21: (no value), wirepad:SMD2
- added IC3: (no value), TI:TL431-ASA
- added R41: 100k, rcl:R-EU_R1206
- added T3: BC847, transistor:BC847
- added T7: IPD50R380, miscrel:IPD50R380
- C3: value 22uF/50V -> 47uF/50V
- C5: value 470p/50V -> 1n/50V; device rcl:C-EUC1206 -> rcl:C-EUC0603
- D10: value 1n4002 -> 20V; device diode:DIODE-DO214AC -> diode:ZENER-DIODESOD80C
- D11: value 1n4002 -> 18V; device diode:DIODE-DO214AC -> diode:ZENER-DIODESOD80C
- L1: value CDRH104R -> 68uH
- R28: value 1M -> 47k
- R39: value 86k -> 22k
- R4, R5: value 1R -> 0.4R
- R40: value 47k -> 20k; device rcl:R-EU_R0805 -> rcl:R-EU_R1206
- R6: value 470k -> 100k
- R7: value 15k -> 12k
Connections:
- removed net N$41: D10.A, D11.C
- removed net N$44: D11.A, R38.1, R39.2
- new net GNDA: C7.2, C9.-, D11.A, D4.A, D6.A, IC2P.V-, PAD10.P, R23.2, R40.1, R9.2, T3.E, T7.S
- new net N$42: D10.A, T3.B
- new net N$43: IC3.K, IC3.R, PAD14.P, R38.1, R6.E
- net GND: now also C2.2, IC3.A, T7.D; no longer C13.-, C2.1, C7.2, C9.-, D10.C, D4.A, D6.A, IC2P.V-, PAD10.P, PAD21.P, R23.2, R9.2
- net N$11: no longer C13.+
- net N$2: now also D11.C, R41.1, T3.C, T7.G; no longer C12.+, IC1.CSP, IC1.VI, PAD12.P, PAD20.P, R2.2, R38.2, R4.2, R5.2, S1.S
- net N$40: now also D10.C, R40.2; no longer PAD14.P, R6.E
- net N$5: now also C2.1; no longer C2.2
- net V+: now also C12.+, IC1.CSP, IC1.VI, PAD12.P, PAD20.P, R2.2, R38.2, R39.2, R4.2, R41.2, R5.2, S1.S
Other:
- note added: "0..1.23V dimming regulation"
- note added: "3x10M opcjonalnie, kondensator moze sie rozladowac przez uplywnosci diod i zasilacz"
- note added: "42V -> 20V nastepuje aktywacja zabezpieczenia przeciw napieciom >42V, ktore spalilyby kontroler LED"
- note added: "Bezpieczna pojemnosc dla Iled_pp <10mA -obliczeniowa C=18uF"
- note added: "OFF<0.5V ON>1.7..Vcc"
- note added: "Rsns=0.2R -> I~1A"
- note added: "Vcc up to 42V"
- note added: "dla 220uH i 36Vo, aby zachowac Irip_pp=24mA Rsns musi nie przekraczac 0.34R, co daje Imax=0,8A dla 51uH I~3A Rsns<0.1R dla 22uH I~1.5A Rsns~0.2R"
- note added: "filter RC"
- note added: "fs = 111kHz"
- note added: "obliczoniowo Cin~18uF dla Vin_pp<1V i Iled~1A (111kHz)"
- note added: "przy odlaczeniu linia GND wskakuje na potencjal V>42"
- note removed: "3x10M opcjonalnie, kondensator moze się rozladowac przez uplywnosci diod i zasilacz"
- note removed: "TO Vcc !!!!"
- note removed: "powinno byc max 47k"
- note removed: "sprawdz podlaczenie radiatora tegoz tyrystora teraz niepodlaczony"
- moved on the sheet: 0R, C1, C12, C2, C3, C5, D1, IC1, L1, PAD12, PAD13, PAD14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
